File: PowerBricksBoard1_X14.brd (EAGLE design)
At the start: 74.9 x 50.8 mm, 16 parts

Commit message: imported new connector into drawing
Parts:
- U$1: value BRICK2DIST -> PETC-02-40-01-X-VT(BTOD); device Brick_Dist_Connector:BRICK2DIST_D2 -> CONN, Distribution-Bricks:SAMTEC_PETC-02-40-01-X-VT_BTOD
- moved H4 165.2 mm to (-67.3, 94.0)
- moved R5 163.7 mm to (-87.6, 91.4), turned to 0 degrees
- moved R4 156.8 mm to (-83.8, 91.4), turned to 0 degrees
- moved R3 155.6 mm to (-80.0, 91.4), turned to 0 degrees
- moved H2 131.8 mm to (-52.1, 94.0)
- moved D1 131.6 mm to (-91.4, 91.4)
- moved R1 131.4 mm to (-72.4, 91.4), turned to 0 degrees
- moved D2 128.7 mm to (-95.2, 91.4)
- moved U$1 115.3 mm to (-74.9, 0.00)
- moved H3 110.3 mm to (-59.7, 94.0)
- moved C1 106.8 mm to (-80.0, 58.4), turned to 0 degrees
- moved R2 101.7 mm to (-76.2, 91.4), flipped to the top, turned to 0 degrees
- moved U$2 94.1 mm to (-68.6, 63.5)
- moved C2 87.9 mm to (-20.3, 95.2), turned to 0 degrees
- moved C4 80.6 mm to (-34.3, 95.2), turned to 0 degrees
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Connections:
- new net 12VGND: U$1.P03_1, U$1.P03_2, U$1.P03_3, U$1.P03_4, U$1.P03_5, U$1.P03_6, U$1.P03_7, U$1.P03_8, U$1.P04_1, U$1.P04_2, U$1.P04_3, U$1.P04_4, U$1.P04_5, U$1.P04_6, U$1.P04_7, U$1.P04_8
- new net 48VGND: U$1.01, U$1.02, U$1.03, U$1.04, U$1.05, U$1.06, U$1.07, U$1.08, U$1.09, U$1.10, U$1.11, U$1.12
- net 12V: now also U$1.P01_1, U$1.P01_2, U$1.P01_3, U$1.P01_4, U$1.P01_5, U$1.P01_6, U$1.P01_7, U$1.P01_8, U$1.P02_1, U$1.P02_2, U$1.P02_3, U$1.P02_4, U$1.P02_5, U$1.P02_6, U$1.P02_7, U$1.P02_8; no longer U$1.2@1, U$1.2@10, U$1.2@11, U$1.2@12, U$1.2@13, U$1.2@14, U$1.2@15, U$1.2@16, U$1.2@17, U$1.2@18, U$1.2@19, U$1.2@2, U$1.2@20, U$1.2@3, U$1.2@4, U$1.2@5, U$1.2@6, U$1.2@7, U$1.2@8, U$1.2@9
- net 12_GND: no longer U$1.4@1, U$1.4@10, U$1.4@11, U$1.4@12, U$1.4@13, U$1.4@14, U$1.4@15, U$1.4@16, U$1.4@17, U$1.4@18, U$1.4@19, U$1.4@2, U$1.4@20, U$1.4@3, U$1.4@4, U$1.4@5, U$1.4@6, U$1.4@7, U$1.4@8, U$1.4@9
- net 48V: now also U$1.29, U$1.30, U$1.31, U$1.32, U$1.33, U$1.34, U$1.35, U$1.36, U$1.37, U$1.38, U$1.39, U$1.40
- net 48V_GND: no longer U$1.1@1, U$1.1@10, U$1.1@2, U$1.1@3, U$1.1@4, U$1.1@5, U$1.1@6, U$1.1@7, U$1.1@8, U$1.1@9
- net 48_GND: no longer U$1.3@1, U$1.3@10, U$1.3@2, U$1.3@3, U$1.3@4, U$1.3@5, U$1.3@6, U$1.3@7, U$1.3@8, U$1.3@9
- net ALERT: now also U$1.17; no longer U$1.D
- net C2: now also U$1.18; no longer U$1.A
- net CLK: now also U$1.19; no longer U$1.C
- net DATA: now also U$1.20; no longer U$1.E
- net ON/OFF: now also U$1.21; no longer U$1.B
Routing:
- net ON/OFF: track 125.6 -> 0.00 mm, vias 1 -> 0
- net N$2: track 41.4 -> 0.00 mm, vias 1 -> 0
- net N$1: track 31.0 -> 0.00 mm
- net ADDR0: track 12.6 -> 0.00 mm
- net C2: track 12.5 -> 0.00 mm
- net DGND: track 9.25 -> 0.00 mm
- net DATA: track 8.99 -> 0.00 mm, vias 1 -> 0
- net ADDR1: track 7.38 -> 0.00 mm
- net ALERT: track 4.58 -> 0.00 mm
- net TRIM: track 4.41 -> 0.00 mm, vias 1 -> 0
- net CLK: track 4.37 -> 0.00 mm
- net 12_GND: track 2.38 -> 0.00 mm, vias 13 -> 0
- net 48_GND: track 1.63 -> 0.00 mm, vias 16 -> 0
- removed copper zone on layer 1, net 12V
- removed copper zone on layer 16, net 12V
- removed copper zone on layer 1, net 12_GND
- removed copper zone on layer 16, net 12_GND
- removed copper zone on layer 1, net 48V_GND
- removed copper zone on layer 16, net 48V_GND
- removed copper zone on layer 1, net 48_GND
- removed copper zone on layer 16, net 48_GND
Other:
- board size 74.9 x 50.8 mm -> 160 x 100 mm
- board text removed: "12V"
- board text removed: "48V"
- board text removed: "=^..^="
- board text removed: "ADDR1 = R3 Resistor ADDR0 = R4 Resistor Octal Address = 8*ADDR1 + ADDR0 0-12 and 40, 44, 45, and 55 address can’t be used (decimal)"
- board text removed: "Octal digit -> Resistor(Kohm) _________ 0 | 10 1 | 15.4 2 | 23.7 3 | 36.5 4 | 54.9 5 | 84.5 6 | 130 7 | 200"
- board text removed: "ROV X13 Power Bricks Board v1 Erin Park Read Hedl Grant Geyer 1-11-2020"
- board text removed: "Trim up: 5.11 * 12 (100+ Delta )/(1.225* Delta) - 511/Delta - 10.2 = resistor to use in kOhm Where Delta is the % up for trim (10% = 10)"
- board text removed: "~(^._.)"

Commit message: Board Size
Parts:
- moved U$2 101.6 mm to (33.0, 62.2)
Other:
- board size 160 x 100 mm -> 76.2 x 50.8 mm
Changed lines of the file:
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@@
 <?xml version="1.0" encoding="utf-8"?>
 <!DOCTYPE eagle SYSTEM "eagle.dtd">
-<eagle version="9.6.2">
+<eagle version="9.5.0">
 <drawing>
 <settings>
@@
 <board>
 <plain>
-<wire x1="0" y1="0" x2="160" y2="0" width="0" layer="20"/>
-<wire x1="160" y1="0" x2="160" y2="100" width="0" layer="20"/>
-<wire x1="160" y1="100" x2="0" y2="100" width="0" layer="20"/>
-<wire x1="0" y1="100" x2="0" y2="0" width="0" layer="20"/>
+<wire x1="0" y1="0" x2="76.2" y2="0" width="0" layer="20"/>
+<wire x1="76.2" y1="0" x2="76.2" y2="50.8" width="0" layer="20"/>
+<wire x1="76.2" y1="50.8" x2="0" y2="50.8" width="0" layer="20"/>
+<wire x1="0" y1="50.8" x2="0" y2="0" width="0" layer="20"/>
 </plain>
 <attributes>
@@
 <attribute name="VALUE" x="-87.63" y="90.678" size="0.6096" layer="27" font="vector" ratio="20" align="top-center"/>
 </element>
-<element name="U$2" library="Delta Power Bricks - Q48SC12050NRDH" package="Q48SC12050NRDH" package3d_urn="urn:adsk.eagle:package:24241038/2" value="Q48SC12050NRDH" x="-68.58" y="63.5" smashed="yes"/>
+<element name="U$2" library="Delta Power Bricks - Q48SC12050NRDH" package="Q48SC12050NRDH" package3d_urn="urn:adsk.eagle:package:24241038/2" value="Q48SC12050NRDH" x="33.02" y="62.23" smashed="yes"/>
 <element name="U$1" library="CONN, Distribution-Bricks" package="SAMTEC_PETC-02-40-01-X-VT_BTOD" value="PETC-02-40-01-X-VT(BTOD)" x="-74.93" y="0" smashed="yes">
 <attribute name="NAME" x="-95.96" y="-1.89" size="1.27" layer="25"/>
@@
 <contactref element="D2" pad="C"/>
 <contactref element="U$2" pad="4"/>
+<wire x1="-16.12" y1="95.25" x2="33.02" y2="77.47" width="0" layer="19" extent="1-1"/>
 <wire x1="-30.09" y1="95.25" x2="-16.12" y2="95.25" width="0" layer="19" extent="1-1"/>
-<wire x1="-68.58" y1="78.74" x2="-30.09" y2="95.25" width="0" layer="19" extent="1-1"/>
-<wire x1="-75.81" y1="58.42" x2="-68.58" y2="78.74" width="0" layer="19" extent="1-1"/>
-<wire x1="-94.373" y1="91.44" x2="-68.58" y2="78.74" width="0" layer="19" extent="1-1"/>
+<wire x1="-75.81" y1="58.42" x2="-30.09" y2="95.25" width="0" layer="19" extent="1-1"/>
+<wire x1="-94.373" y1="91.44" x2="-75.81" y2="58.42" width="0" layer="19" extent="1-1"/>
 </signal>
 <signal name="12V">
@@
 <contactref element="U$1" pad="P02_4"/>
 <contactref element="U$1" pad="P02_6"/>
+<wire x1="83.82" y1="62.23" x2="83.82" y2="66.04" width="0" layer="19" extent="1-1"/>
+<wire x1="-36.195" y1="-5.08" x2="83.82" y2="62.23" width="0" layer="19" extent="1-1"/>
+<wire x1="-38.735" y1="-5.08" x2="-36.195" y2="-5.08" width="0" layer="19" extent="1-1"/>
+<wire x1="-38.735" y1="-7.62" x2="-38.735" y2="-5.08" width="0" layer="19" extent="1-1"/>
+<wire x1="-38.735" y1="-10.16" x2="-38.735" y2="-7.62" width="0" layer="19" extent="1-1"/>
+<wire x1="-38.735" y1="-12.7" x2="-38.735" y2="-10.16" width="0" layer="19" extent="1-1"/>
+<wire x1="-36.195" y1="-12.7" x2="-38.735" y2="-12.7" width="0" layer="19" extent="1-1"/>
+<wire x1="-36.195" y1="-10.16" x2="-38.735" y2="-10.16" width="0" layer="19" extent="1-1"/>
+<wire x1="-36.195" y1="-7.62" x2="-36.195" y2="-5.08" width="0" layer="19" extent="1-1"/>
+<wire x1="-42.545" y1="-12.7" x2="-38.735" y2="-12.7" width="0" layer="19" extent="1-1"/>
+<wire x1="-45.085" y1="-12.7" x2="-42.545" y2="-12.7" width="0" layer="19" extent="1-1"/>
 <wire x1="-45.085" y1="-10.16" x2="-45.085" y2="-12.7" width="0" layer="19" extent="1-1"/>
-<wire x1="-42.545" y1="-12.7" x2="-45.085" y2="-12.7" width="0" layer="19" extent="1-1"/>
-<wire x1="-42.545" y1="-10.16" x2="-45.085" y2="-10.16" width="0" layer="19" extent="1-1"/>
+<wire x1="-42.545" y1="-10.16" x2="-42.545" y2="-12.7" width="0" layer="19" extent="1-1"/>
 <wire x1="-45.085" y1="-7.62" x2="-45.085" y2="-10.16" width="0" layer="19" extent="1-1"/>
 <wire x1="-45.085" y1="-5.08" x2="-45.085" y2="-7.62" width="0" layer="19" extent="1-1"/>
 <wire x1="-42.545" y1="-7.62" x2="-42.545" y2="-10.16" width="0" layer="19" extent="1-1"/>
 <wire x1="-42.545" y1="-5.08" x2="-45.085" y2="-5.08" width="0" layer="19" extent="1-1"/>
-<wire x1="-38.735" y1="-12.7" x2="-42.545" y2="-12.7" width="0" layer="19" extent="1-1"/>
-<wire x1="-38.735" y1="-10.16" x2="-38.735" y2="-12.7" width="0" layer="19" extent="1-1"/>
-<wire x1="-36.195" y1="-12.7" x2="-38.735" y2="-12.7" width="0" layer="19" extent="1-1"/>
-<wire x1="-36.195" y1="-10.16" x2="-38.735" y2="-10.16" width="0" layer="19" extent="1-1"/>
-<wire x1="-38.735" y1="-7.62" x2="-38.735" y2="-10.16" width="0" layer="19" extent="1-1"/>
-<wire x1="-38.735" y1="-5.08" x2="-38.735" y2="-7.62" width="0" layer="19" extent="1-1"/>
-<wire x1="-36.195" y1="-7.62" x2="-36.195" y2="-10.16" width="0" layer="19" extent="1-1"/>
-<wire x1="-36.195" y1="-5.08" x2="-38.735" y2="-5.08" width="0" layer="19" extent="1-1"/>
-<wire x1="-17.78" y1="63.5" x2="-36.195" y2="-5.08" width="0" layer="19" extent="1-1"/>
-<wire x1="-17.78" y1="67.31" x2="-17.78" y2="63.5" width="0" layer="19" extent="1-1"/>
-<wire x1="-71.54" y1="91.44" x2="-17.78" y2="67.31" width="0" layer="19" extent="1-1"/>
+<wire x1="-71.54" y1="91.44" x2="-45.085" y2="-5.08" width="0" layer="19" extent="1-1"/>
 <wire x1="-86.78" y1="91.44" x2="-71.54" y2="91.44" width="0" layer="19" extent="1-1"/>
 </signal>
@@
 <contactref element="U$2" pad="10"/>
 <contactref element="U$1" pad="18"/>
-<wire x1="-15.24" y1="77.12" x2="-59.69" y2="-10.16" width="0" layer="19" extent="1-1"/>
+<wire x1="-59.69" y1="-10.16" x2="86.36" y2="75.85" width="0" layer="19" extent="1-1"/>
 </signal>
 <signal name="12_GND">
@@
 <contactref element="U$2" pad="5"/>
 <contactref element="U$2" pad="6"/>
-<wire x1="-17.78" y1="74.93" x2="-17.78" y2="78.74" width="0" layer="19" extent="1-1"/>
-<wire x1="-90.563" y1="91.44" x2="-17.78" y2="78.74" width="0" layer="19" extent="1-1"/>
+<wire x1="83.82" y1="73.66" x2="83.82" y2="77.47" width="0" layer="19" extent="1-1"/>
+<wire x1="-90.563" y1="91.44" x2="83.82" y2="77.47" width="0" layer="19" extent="1-1"/>
 </signal>
 <signal name="ALERT">
 <contactref element="U$2" pad="13"/>
 <contactref element="U$1" pad="17"/>
-<wire x1="-15.24" y1="71.12" x2="-59.69" y2="-12.7" width="0" layer="19" extent="1-1"/>
+<wire x1="-59.69" y1="-12.7" x2="86.36" y2="69.85" width="0" layer="19" extent="1-1"/>
 </signal>
 <signal name="DATA">
 <contactref element="U$2" pad="12"/>
 <contactref element="U$1" pad="20"/>
-<wire x1="-15.24" y1="73.12" x2="-59.69" y2="-5.08" width="0" layer="19" extent="1-1"/>
+<wire x1="-59.69" y1="-5.08" x2="86.36" y2="71.85" width="0" layer="19" extent="1-1"/>
 </signal>
 <signal name="CLK">
 <contactref element="U$2" pad="14"/>
 <contactref element="U$1" pad="19"/>
-<wire x1="-15.24" y1="69.12" x2="-59.69" y2="-7.62" width="0" layer="19" extent="1-1"/>
+<wire x1="-59.69" y1="-7.62" x2="86.36" y2="67.85" width="0" layer="19" extent="1-1"/>
 </signal>
 <signal name="N$1">
@@
 <contactref element="R3" pad="1"/>
 <contactref element="U$2" pad="11"/>
-<wire x1="-80.86" y1="91.44" x2="-15.24" y2="75.12" width="0" layer="19" extent="1-1"/>
+<wire x1="-80.86" y1="91.44" x2="86.36" y2="73.85" width="0" layer="19" extent="1-1"/>
 <wire x1="-84.67" y1="91.44" x2="-80.86" y2="91.44" width="0" layer="19" extent="1-1"/>
 </signal>
@@
 <contactref element="R3" pad="2"/>
 <contactref element="U$2" pad="15"/>
-<wire x1="-79.16" y1="91.44" x2="-15.24" y2="67.12" width="0" layer="19" extent="1-1"/>
+<wire x1="-79.16" y1="91.44" x2="86.36" y2="65.85" width="0" layer="19" extent="1-1"/>
 </signal>
 <signal name="ADDR0">
 <contactref element="U$2" pad="16"/>
 <contactref element="R4" pad="2"/>
-<wire x1="-82.97" y1="91.44" x2="-15.24" y2="65.12" width="0" layer="19" extent="1-1"/>
+<wire x1="-82.97" y1="91.44" x2="86.36" y2="63.85" width="0" layer="19" extent="1-1"/>
 </signal>
 <signal name="TRIM">
 <contactref element="R5" pad="1"/>
 <contactref element="U$2" pad="7"/>
-<wire x1="-88.48" y1="91.44" x2="-17.78" y2="71.12" width="0" layer="19" extent="1-1"/>
+<wire x1="-88.48" y1="91.44" x2="83.82" y2="69.85" width="0" layer="19" extent="1-1"/>
 </signal>
 <signal name="ON/OFF">
 <contactref element="U$2" pad="2"/>
 <contactref element="U$1" pad="21"/>
-<wire x1="-68.58" y1="71.12" x2="-62.23" y2="-12.7" width="0" layer="19" extent="1-1"/>
+<wire x1="-62.23" y1="-12.7" x2="33.02" y2="69.85" width="0" layer="19" extent="1-1"/>
 </signal>
 <signal name="48V">

Commit message: Update PowerBricksBoard1_X14.brd
Parts:
- moved U$2 50.7 mm to (14.0, 15.2)
Changed lines of the file:
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@@
 <?xml version="1.0" encoding="utf-8"?>
 <!DOCTYPE eagle SYSTEM "eagle.dtd">
-<eagle version="9.5.0">
+<eagle version="9.6.2">
 <drawing>
 <settings>
@@
 <attribute name="VALUE" x="-87.63" y="90.678" size="0.6096" layer="27" font="vector" ratio="20" align="top-center"/>
 </element>
-<element name="U$2" library="Delta Power Bricks - Q48SC12050NRDH" package="Q48SC12050NRDH" package3d_urn="urn:adsk.eagle:package:24241038/2" value="Q48SC12050NRDH" x="33.02" y="62.23" smashed="yes"/>
+<element name="U$2" library="Delta Power Bricks - Q48SC12050NRDH" package="Q48SC12050NRDH" package3d_urn="urn:adsk.eagle:package:24241038/2" value="Q48SC12050NRDH" x="13.97" y="15.24" smashed="yes"/>
 <element name="U$1" library="CONN, Distribution-Bricks" package="SAMTEC_PETC-02-40-01-X-VT_BTOD" value="PETC-02-40-01-X-VT(BTOD)" x="-74.93" y="0" smashed="yes">
 <attribute name="NAME" x="-95.96" y="-1.89" size="1.27" layer="25"/>
@@
 <contactref element="D2" pad="C"/>
 <contactref element="U$2" pad="4"/>
-<wire x1="-16.12" y1="95.25" x2="33.02" y2="77.47" width="0" layer="19" extent="1-1"/>
+<wire x1="-16.12" y1="95.25" x2="13.97" y2="30.48" width="0" layer="19" extent="1-1"/>
 <wire x1="-30.09" y1="95.25" x2="-16.12" y2="95.25" width="0" layer="19" extent="1-1"/>
 <wire x1="-75.81" y1="58.42" x2="-30.09" y2="95.25" width="0" layer="19" extent="1-1"/>
@@
 <contactref element="U$1" pad="P02_4"/>
 <contactref element="U$1" pad="P02_6"/>
-<wire x1="83.82" y1="62.23" x2="83.82" y2="66.04" width="0" layer="19" extent="1-1"/>
-<wire x1="-36.195" y1="-5.08" x2="83.82" y2="62.23" width="0" layer="19" extent="1-1"/>
+<wire x1="64.77" y1="15.24" x2="64.77" y2="19.05" width="0" layer="19" extent="1-1"/>
+<wire x1="-36.195" y1="-5.08" x2="64.77" y2="15.24" width="0" layer="19" extent="1-1"/>
 <wire x1="-38.735" y1="-5.08" x2="-36.195" y2="-5.08" width="0" layer="19" extent="1-1"/>
 <wire x1="-38.735" y1="-7.62" x2="-38.735" y2="-5.08" width="0" layer="19" extent="1-1"/>
@@
 <contactref element="U$2" pad="10"/>
 <contactref element="U$1" pad="18"/>
-<wire x1="-59.69" y1="-10.16" x2="86.36" y2="75.85" width="0" layer="19" extent="1-1"/>
+<wire x1="-59.69" y1="-10.16" x2="67.31" y2="28.86" width="0" layer="19" extent="1-1"/>
 </signal>
 <signal name="12_GND">
@@
 <contactref element="U$2" pad="5"/>
 <contactref element="U$2" pad="6"/>
-<wire x1="83.82" y1="73.66" x2="83.82" y2="77.47" width="0" layer="19" extent="1-1"/>
-<wire x1="-90.563" y1="91.44" x2="83.82" y2="77.47" width="0" layer="19" extent="1-1"/>
+<wire x1="64.77" y1="26.67" x2="64.77" y2="30.48" width="0" layer="19" extent="1-1"/>
+<wire x1="-90.563" y1="91.44" x2="64.77" y2="30.48" width="0" layer="19" extent="1-1"/>
 </signal>
 <signal name="ALERT">
 <contactref element="U$2" pad="13"/>
 <contactref element="U$1" pad="17"/>
-<wire x1="-59.69" y1="-12.7" x2="86.36" y2="69.85" width="0" layer="19" extent="1-1"/>
+<wire x1="-59.69" y1="-12.7" x2="67.31" y2="22.86" width="0" layer="19" extent="1-1"/>
 </signal>
 <signal name="DATA">
 <contactref element="U$2" pad="12"/>
 <contactref element="U$1" pad="20"/>
-<wire x1="-59.69" y1="-5.08" x2="86.36" y2="71.85" width="0" layer="19" extent="1-1"/>
+<wire x1="-59.69" y1="-5.08" x2="67.31" y2="24.86" width="0" layer="19" extent="1-1"/>
 </signal>
 <signal name="CLK">
 <contactref element="U$2" pad="14"/>
 <contactref element="U$1" pad="19"/>
-<wire x1="-59.69" y1="-7.62" x2="86.36" y2="67.85" width="0" layer="19" extent="1-1"/>
+<wire x1="-59.69" y1="-7.62" x2="67.31" y2="20.86" width="0" layer="19" extent="1-1"/>
 </signal>
 <signal name="N$1">
@@
 <contactref element="R3" pad="1"/>
 <contactref element="U$2" pad="11"/>
-<wire x1="-80.86" y1="91.44" x2="86.36" y2="73.85" width="0" layer="19" extent="1-1"/>
+<wire x1="-80.86" y1="91.44" x2="67.31" y2="26.86" width="0" layer="19" extent="1-1"/>
 <wire x1="-84.67" y1="91.44" x2="-80.86" y2="91.44" width="0" layer="19" extent="1-1"/>
 </signal>
@@
 <contactref element="R3" pad="2"/>
 <contactref element="U$2" pad="15"/>
-<wire x1="-79.16" y1="91.44" x2="86.36" y2="65.85" width="0" layer="19" extent="1-1"/>
+<wire x1="-79.16" y1="91.44" x2="67.31" y2="18.86" width="0" layer="19" extent="1-1"/>
 </signal>
 <signal name="ADDR0">
 <contactref element="U$2" pad="16"/>
 <contactref element="R4" pad="2"/>
-<wire x1="-82.97" y1="91.44" x2="86.36" y2="63.85" width="0" layer="19" extent="1-1"/>
+<wire x1="-82.97" y1="91.44" x2="67.31" y2="16.86" width="0" layer="19" extent="1-1"/>
 </signal>
 <signal name="TRIM">
 <contactref element="R5" pad="1"/>
 <contactref element="U$2" pad="7"/>
-<wire x1="-88.48" y1="91.44" x2="83.82" y2="69.85" width="0" layer="19" extent="1-1"/>
+<wire x1="-88.48" y1="91.44" x2="64.77" y2="22.86" width="0" layer="19" extent="1-1"/>
 </signal>
 <signal name="ON/OFF">
 <contactref element="U$2" pad="2"/>
 <contactref element="U$1" pad="21"/>
-<wire x1="-62.23" y1="-12.7" x2="33.02" y2="69.85" width="0" layer="19" extent="1-1"/>
+<wire x1="-62.23" y1="-12.7" x2="13.97" y2="22.86" width="0" layer="19" extent="1-1"/>
 </signal>
 <signal name="48V">

Commit message: update
Parts:
- moved R5 177.2 mm to (72.4, 15.2)
- moved D2 177.1 mm to (72.4, 34.3)
- moved D1 172.7 mm to (72.4, 36.8)
- moved R4 172.2 mm to (72.4, 19.1)
- moved R3 167.1 mm to (72.4, 22.9)
- moved R2 162.1 mm to (72.4, 26.7)
- moved H3 159.9 mm to (72.4, 3.81)
- moved R1 157.1 mm to (72.4, 30.5)
- moved H4 147.4 mm to (72.4, 47.0)
- moved H2 106.1 mm to (3.81, 3.81)
- moved C1 102.6 mm to (20.3, 36.8), turned to 90 degrees
- moved U$1 102.0 mm to (24.1, 24.1)
- moved C4 88.2 mm to (31.8, 36.8), turned to 90 degrees
- moved C2 86.3 mm to (43.2, 36.8), turned to 90 degrees
- moved H1 67.4 mm to (3.81, 47.0)
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Connections:
- removed net 48V_GND: U$2.1
- net 48V: now also U$2.1
Routing:
- net 48_GND: track 0.00 -> 8.31 mm
